File: Pi5-Artix50T-Hat.kicad_pcb (KiCad board)
At the start: 2 copper layers, 65 x 56 mm, 5 parts, among them J1 GPIO

Commit message: Schematic finished, starting layout
Parts:
- added C1: 100n, Capacitor_SMD:C_0402_1005Metric_Pad0.74x0.62mm_HandSolder, F.Cu at (-50.0, 134.1)
- added C10: 4.7u, Capacitor_SMD:C_0402_1005Metric_Pad0.74x0.62mm_HandSolder, F.Cu at (33.7, -10.5)
- added C100: 100u, Capacitor_SMD:C_1206_3216Metric_Pad1.33x1.80mm_HandSolder, F.Cu at (-41.6, 115.0)
- added C11: 100n, Capacitor_SMD:C_0402_1005Metric_Pad0.74x0.62mm_HandSolder, F.Cu at (33.7, -8.52)
- added C12: 100n, Capacitor_SMD:C_0402_1005Metric_Pad0.74x0.62mm_HandSolder, F.Cu at (33.7, -6.55)
- added C13: 100n, Capacitor_SMD:C_0402_1005Metric_Pad0.74x0.62mm_HandSolder, F.Cu at (36.5, 3.33)
- added C14: 4.7u, Capacitor_SMD:C_0402_1005Metric_Pad0.74x0.62mm_HandSolder, F.Cu at (-49.4, 3.94)
- added C15: 4.7u, Capacitor_SMD:C_0402_1005Metric_Pad0.74x0.62mm_HandSolder, F.Cu at (33.7, -4.58)
- added C16: 4.7u, Capacitor_SMD:C_0402_1005Metric_Pad0.74x0.62mm_HandSolder, F.Cu at (-49.4, 5.91)
- added C17: 4.7u, Capacitor_SMD:C_0402_1005Metric_Pad0.74x0.62mm_HandSolder, F.Cu at (-49.4, 7.88)
- added C18: 4.7n, Capacitor_SMD:C_0402_1005Metric_Pad0.74x0.62mm_HandSolder, F.Cu at (-49.4, 9.85)
- added C19: 100n, Capacitor_SMD:C_0402_1005Metric_Pad0.74x0.62mm_HandSolder, F.Cu at (36.5, 5.30)
- added C2: 100n, Capacitor_SMD:C_0402_1005Metric_Pad0.74x0.62mm_HandSolder, F.Cu at (120.9, 79.5)
- added C20: 4.7u, Capacitor_SMD:C_0402_1005Metric_Pad0.74x0.62mm_HandSolder, F.Cu at (-49.4, 25.0)
- added C21: 4.7u, Capacitor_SMD:C_0402_1005Metric_Pad0.74x0.62mm_HandSolder, F.Cu at (-49.4, 27.0)
- added C22: 4.7u, Capacitor_SMD:C_0402_1005Metric_Pad0.74x0.62mm_HandSolder, F.Cu at (-49.4, 28.9)
- added C23: 4.7u, Capacitor_SMD:C_0402_1005Metric_Pad0.74x0.62mm_HandSolder, F.Cu at (-49.4, 30.9)
- added C24: 4.7n, Capacitor_SMD:C_0402_1005Metric_Pad0.74x0.62mm_HandSolder, F.Cu at (-49.4, 32.9)
- added C25: 4.7u, Capacitor_SMD:C_0402_1005Metric_Pad0.74x0.62mm_HandSolder, F.Cu at (-49.4, 34.9)
- added C26: 4.7u, Capacitor_SMD:C_0402_1005Metric_Pad0.74x0.62mm_HandSolder, F.Cu at (36.5, 7.27)
- added C27: 4.7u, Capacitor_SMD:C_0402_1005Metric_Pad0.74x0.62mm_HandSolder, F.Cu at (-50.4, 50.0)
- added C28: 4.7u, Capacitor_SMD:C_0402_1005Metric_Pad0.74x0.62mm_HandSolder, F.Cu at (-50.4, 52.0)
- added C29: 4.7u, Capacitor_SMD:C_0402_1005Metric_Pad0.74x0.62mm_HandSolder, F.Cu at (-50.4, 53.9)
- added C3: 100n, Capacitor_SMD:C_0402_1005Metric_Pad0.74x0.62mm_HandSolder, F.Cu at (120.9, 78.5)
- added C30: 4.7u, Capacitor_SMD:C_0402_1005Metric_Pad0.74x0.62mm_HandSolder, F.Cu at (-50.4, 55.9)
- added C31: 3.3n, Capacitor_SMD:C_0402_1005Metric_Pad0.74x0.62mm_HandSolder, F.Cu at (-50.4, 57.9)
- added C32: 4.7u, Capacitor_SMD:C_0402_1005Metric_Pad0.74x0.62mm_HandSolder, F.Cu at (-50.4, 59.9)
- added C33: 100n, Capacitor_SMD:C_0402_1005Metric_Pad0.74x0.62mm_HandSolder, F.Cu at (15.0, 25.0)
- added C34: 4.7u, Capacitor_SMD:C_0402_1005Metric_Pad0.74x0.62mm_HandSolder, F.Cu at (-50.0, 75.0)
- added C35: 4.7u, Capacitor_SMD:C_0402_1005Metric_Pad0.74x0.62mm_HandSolder, F.Cu at (-50.0, 77.0)
- added C36: 4.7u, Capacitor_SMD:C_0402_1005Metric_Pad0.74x0.62mm_HandSolder, F.Cu at (-50.0, 78.9)
- added C37: 4.7u, Capacitor_SMD:C_0402_1005Metric_Pad0.74x0.62mm_HandSolder, F.Cu at (-50.0, 80.9)
- added C38: 1.5n, Capacitor_SMD:C_0402_1005Metric_Pad0.74x0.62mm_HandSolder, F.Cu at (-50.0, 82.9)
- added C39: 4.7u, Capacitor_SMD:C_0402_1005Metric_Pad0.74x0.62mm_HandSolder, F.Cu at (-50.0, 84.8)
- added C4: 100n, Capacitor_SMD:C_0402_1005Metric_Pad0.74x0.62mm_HandSolder, F.Cu at (30.5, -6.55)
- added C40: 100n, Capacitor_SMD:C_0402_1005Metric_Pad0.74x0.62mm_HandSolder, F.Cu at (15.0, 27.0)
- added C41: 4.7u, Capacitor_SMD:C_0402_1005Metric_Pad0.74x0.62mm_HandSolder, F.Cu at (-49.4, 100.0)
- added C42: 4.7u, Capacitor_SMD:C_0402_1005Metric_Pad0.74x0.62mm_HandSolder, F.Cu at (-49.4, 102.0)
- added C43: 4.7u, Capacitor_SMD:C_0402_1005Metric_Pad0.74x0.62mm_HandSolder, F.Cu at (-49.4, 103.9)
- added C44: 4.7u, Capacitor_SMD:C_0402_1005Metric_Pad0.74x0.62mm_HandSolder, F.Cu at (-49.4, 105.9)
- added C45: 2.7n, Capacitor_SMD:C_0402_1005Metric_Pad0.74x0.62mm_HandSolder, F.Cu at (-49.4, 107.9)
- added C46: 4.7u, Capacitor_SMD:C_0402_1005Metric_Pad0.74x0.62mm_HandSolder, F.Cu at (-49.4, 109.8)
- added C47: 100n, Capacitor_SMD:C_0402_1005Metric_Pad0.74x0.62mm_HandSolder, F.Cu at (-15.1, 128.0)
- added C48: 4.7u, Capacitor_SMD:C_0402_1005Metric_Pad0.74x0.62mm_HandSolder, F.Cu at (-15.1, 130.0)
- added C49: 10n, Capacitor_SMD:C_0402_1005Metric_Pad0.74x0.62mm_HandSolder, F.Cu at (-49.4, 11.8)
- added C5: 100n, Capacitor_SMD:C_0402_1005Metric_Pad0.74x0.62mm_HandSolder, F.Cu at (30.5, -4.58)
- added C50: 10n, Capacitor_SMD:C_0402_1005Metric_Pad0.74x0.62mm_HandSolder, F.Cu at (-49.4, 36.8)
- added C51: 10n, Capacitor_SMD:C_0402_1005Metric_Pad0.74x0.62mm_HandSolder, F.Cu at (-50.4, 61.8)
- added C52: 10n, Capacitor_SMD:C_0402_1005Metric_Pad0.74x0.62mm_HandSolder, F.Cu at (-50.0, 86.8)
- added C53: 10n, Capacitor_SMD:C_0402_1005Metric_Pad0.74x0.62mm_HandSolder, F.Cu at (-49.4, 111.8)
- added C54: 4.7u, Capacitor_SMD:C_0402_1005Metric_Pad0.74x0.62mm_HandSolder, F.Cu at (15.0, 29.0)
- added C55: 100n, Capacitor_SMD:C_0402_1005Metric_Pad0.74x0.62mm_HandSolder, F.Cu at (15.0, 30.9)
- added C56: 100n, Capacitor_SMD:C_0402_1005Metric_Pad0.74x0.62mm_HandSolder, F.Cu at (15.0, 32.9)
- added C57: 100n, Capacitor_SMD:C_0402_1005Metric_Pad0.74x0.62mm_HandSolder, F.Cu at (18.2, 25.0)
- added C58: 100n, Capacitor_SMD:C_0402_1005Metric_Pad0.74x0.62mm_HandSolder, F.Cu at (30.5, 21.4)
- added C59: 100n, Capacitor_SMD:C_0402_1005Metric_Pad0.74x0.62mm_HandSolder, F.Cu at (18.2, 27.0)
- added C6: 100n, Capacitor_SMD:C_0402_1005Metric_Pad0.74x0.62mm_HandSolder, F.Cu at (120.9, 80.5)
- added C60: 100n, Capacitor_SMD:C_0402_1005Metric_Pad0.74x0.62mm_HandSolder, F.Cu at (18.2, 29.0)
- added C61: 100n, Capacitor_SMD:C_0402_1005Metric_Pad0.74x0.62mm_HandSolder, F.Cu at (18.2, 30.9)
- added C62: 100n, Capacitor_SMD:C_0402_1005Metric_Pad0.74x0.62mm_HandSolder, F.Cu at (18.2, 32.9)
- added C63: 100n, Capacitor_SMD:C_0402_1005Metric_Pad0.74x0.62mm_HandSolder, F.Cu at (21.4, 25.0)
- added C64: 100n, Capacitor_SMD:C_0402_1005Metric_Pad0.74x0.62mm_HandSolder, F.Cu at (21.4, 27.0)
- added C65: 4.7u, Capacitor_SMD:C_0402_1005Metric_Pad0.74x0.62mm_HandSolder, F.Cu at (21.4, 29.0)
- added C66: 100n, Capacitor_SMD:C_0402_1005Metric_Pad0.74x0.62mm_HandSolder, F.Cu at (30.5, 23.4)
- added C67: 100n, Capacitor_SMD:C_0402_1005Metric_Pad0.74x0.62mm_HandSolder, F.Cu at (30.5, 25.3)
- added C68: 100n, Capacitor_SMD:C_0402_1005Metric_Pad0.74x0.62mm_HandSolder, F.Cu at (30.5, 27.3)
- added C69: 100n, Capacitor_SMD:C_0402_1005Metric_Pad0.74x0.62mm_HandSolder, F.Cu at (30.5, 29.3)
- added C7: 100n, Capacitor_SMD:C_0402_1005Metric_Pad0.74x0.62mm_HandSolder, F.Cu at (120.9, 81.5)
- added C70: 100n, Capacitor_SMD:C_0402_1005Metric_Pad0.74x0.62mm_HandSolder, F.Cu at (33.7, 21.4)
- added C71: 4.7u, Capacitor_SMD:C_0402_1005Metric_Pad0.74x0.62mm_HandSolder, F.Cu at (33.7, 23.4)
- added C72: 100n, Capacitor_SMD:C_0402_1005Metric_Pad0.74x0.62mm_HandSolder, F.Cu at (33.7, 25.3)
- added C73: 100n, Capacitor_SMD:C_0402_1005Metric_Pad0.74x0.62mm_HandSolder, F.Cu at (33.7, 27.3)
- added C74: 100n, Capacitor_SMD:C_0402_1005Metric_Pad0.74x0.62mm_HandSolder, F.Cu at (33.7, 29.3)
- added C75: 100n, Capacitor_SMD:C_0402_1005Metric_Pad0.74x0.62mm_HandSolder, F.Cu at (36.9, 21.4)
- added C76: 100n, Capacitor_SMD:C_0402_1005Metric_Pad0.74x0.62mm_HandSolder, F.Cu at (36.9, 23.4)
- added C77: 100n, Capacitor_SMD:C_0402_1005Metric_Pad0.74x0.62mm_HandSolder, F.Cu at (36.9, 25.3)
- added C78: 4.7u, Capacitor_SMD:C_0402_1005Metric_Pad0.74x0.62mm_HandSolder, F.Cu at (36.9, 27.3)
- added C79: 100n, Capacitor_SMD:C_0402_1005Metric_Pad0.74x0.62mm_HandSolder, F.Cu at (3.35, 25.0)
- added C8: 4.7u, Capacitor_SMD:C_0402_1005Metric_Pad0.74x0.62mm_HandSolder, F.Cu at (-49.4, 0.00)
- added C80: 100n, Capacitor_SMD:C_0402_1005Metric_Pad0.74x0.62mm_HandSolder, F.Cu at (3.35, 27.0)
- added C81: 100n, Capacitor_SMD:C_0402_1005Metric_Pad0.74x0.62mm_HandSolder, F.Cu at (3.35, 29.0)
- added C82: 100n, Capacitor_SMD:C_0402_1005Metric_Pad0.74x0.62mm_HandSolder, F.Cu at (3.35, 30.9)
- added C83: 100n, Capacitor_SMD:C_0402_1005Metric_Pad0.74x0.62mm_HandSolder, F.Cu at (3.35, 32.9)
- added C84: 100n, Capacitor_SMD:C_0402_1005Metric_Pad0.74x0.62mm_HandSolder, F.Cu at (6.56, 25.0)
- added C85: 4.7u, Capacitor_SMD:C_0402_1005Metric_Pad0.74x0.62mm_HandSolder, F.Cu at (6.56, 27.0)
- added C86: 100n, Capacitor_SMD:C_0402_1005Metric_Pad0.74x0.62mm_HandSolder, F.Cu at (6.56, 29.0)
- added C87: 100n, Capacitor_SMD:C_0402_1005Metric_Pad0.74x0.62mm_HandSolder, F.Cu at (6.56, 30.9)
- added C88: 100n, Capacitor_SMD:C_0402_1005Metric_Pad0.74x0.62mm_HandSolder, F.Cu at (6.56, 32.9)
- added C89: 100n, Capacitor_SMD:C_0402_1005Metric_Pad0.74x0.62mm_HandSolder, F.Cu at (9.77, 25.0)
- added C9: 4.7u, Capacitor_SMD:C_0402_1005Metric_Pad0.74x0.62mm_HandSolder, F.Cu at (-49.4, 1.97)
- added C90: 100n, Capacitor_SMD:C_0402_1005Metric_Pad0.74x0.62mm_HandSolder, F.Cu at (9.77, 27.0)
- added C91: 100n, Capacitor_SMD:C_0402_1005Metric_Pad0.74x0.62mm_HandSolder, F.Cu at (9.77, 29.0)
- added C92: 4.7u, Capacitor_SMD:C_0402_1005Metric_Pad0.74x0.62mm_HandSolder, F.Cu at (9.77, 30.9)
- added C93: 100n, Capacitor_SMD:C_0402_1005Metric_Pad0.74x0.62mm_HandSolder, F.Cu at (-45.9, 155.3)
- added C94: 4.7u, Capacitor_SMD:C_0402_1005Metric_Pad0.74x0.62mm_HandSolder, F.Cu at (-45.9, 157.3)
- added C95: 100u, Capacitor_SMD:C_1206_3216Metric_Pad1.33x1.80mm_HandSolder, F.Cu at (-39.1, 10.0)
- added C96: 100u, Capacitor_SMD:C_1206_3216Metric_Pad1.33x1.80mm_HandSolder, F.Cu at (-59.1, 20.0)
- added C97: 100u, Capacitor_SMD:C_1206_3216Metric_Pad1.33x1.80mm_HandSolder, F.Cu at (-39.1, 35.0)
- added C98: 100u, Capacitor_SMD:C_1206_3216Metric_Pad1.33x1.80mm_HandSolder, F.Cu at (-39.1, 60.0)
- added C99: 100u, Capacitor_SMD:C_1206_3216Metric_Pad1.33x1.80mm_HandSolder, F.Cu at (-40.9, 85.0)
- added D1: RED, LED_SMD:LED_0603_1608Metric_Pad1.05x0.95mm_HandSolder, F.Cu at (86.6, 90.0)
- added D2: RED, LED_SMD:LED_0603_1608Metric_Pad1.05x0.95mm_HandSolder, F.Cu at (-8.15, 126.6)
- added FB1: 600Ω@100MHz, Inductor_SMD:L_0603_1608Metric_Pad1.05x0.95mm_HandSolder, F.Cu at (37.4, -10.2)
- added FB2: 600Ω@100MHz, Inductor_SMD:L_0603_1608Metric_Pad1.05x0.95mm_HandSolder, F.Cu at (37.4, -7.71)
- added FB3: 600Ω@100MHz, Inductor_SMD:L_0603_1608Metric_Pad1.05x0.95mm_HandSolder, F.Cu at (-49.7, 155.6)
- added J2: Molex 0878321420, Connector_PinHeader_2.00mm:PinHeader_2x07_P2.00mm_Vertical, F.Cu at (-14.5, 145.1)
- added J3: 68711614522, pcie:68711614522, F.Cu at (107.3, 72.0)
- added JP1: ID_WP, Jumper:SolderJumper-2_P1.3mm_Open_TrianglePad1.0x1.5mm, F.Cu at (-49.4, 131.3)
- added JP2: ID_WP, Jumper:SolderJumper-2_P1.3mm_Open_TrianglePad1.0x1.5mm, F.Cu at (-45.7, 9.84)
- added JP3: ID_WP, Jumper:SolderJumper-2_P1.3mm_Open_TrianglePad1.0x1.5mm, F.Cu at (-45.7, 34.8)
- added JP4: ID_WP, Jumper:SolderJumper-2_P1.3mm_Open_TrianglePad1.0x1.5mm, F.Cu at (-46.6, 59.8)
- added JP5: ID_WP, Jumper:SolderJumper-2_P1.3mm_Open_TrianglePad1.0x1.5mm, F.Cu at (-46.2, 84.8)
- added JP6: ID_WP, Jumper:SolderJumper-2_P1.3mm_Open_TrianglePad1.0x1.5mm, F.Cu at (-45.7, 109.8)
- added JP7: ID_WP, Jumper:SolderJumper-2_P1.3mm_Open_TrianglePad1.0x1.5mm, F.Cu at (-36.8, 110.0)
- added R1: 3.9k, Resistor_SMD:R_0402_1005Metric_Pad0.72x0.64mm_HandSolder, F.Cu at (-45.6, 130.5)
- added R10: 330, Resistor_SMD:R_0402_1005Metric_Pad0.72x0.64mm_HandSolder, F.Cu at (30.4, 52.0)
- added R11: 1k, Resistor_SMD:R_0402_1005Metric_Pad0.72x0.64mm_HandSolder, F.Cu at (86.0, 92.3)
- added R12: 1k, Resistor_SMD:R_0402_1005Metric_Pad0.72x0.64mm_HandSolder, F.Cu at (30.4, 56.0)
- added R13: 100, Resistor_SMD:R_0402_1005Metric_Pad0.72x0.64mm_HandSolder, F.Cu at (30.4, 58.0)
- added R14: 0, Resistor_SMD:R_0402_1005Metric_Pad0.72x0.64mm_HandSolder, F.Cu at (-39.8, 0.01)
- added R15: 4.99k, Resistor_SMD:R_0402_1005Metric_Pad0.72x0.64mm_HandSolder, F.Cu at (-39.8, 2.00)
- added R16: 1k, Resistor_SMD:R_0402_1005Metric_Pad0.72x0.64mm_HandSolder, F.Cu at (-39.8, 3.99)
- added R17: 1k, Resistor_SMD:R_0402_1005Metric_Pad0.72x0.64mm_HandSolder, F.Cu at (-39.8, 25.0)
- added R18: 4.99k, Resistor_SMD:R_0402_1005Metric_Pad0.72x0.64mm_HandSolder, F.Cu at (-39.8, 27.0)
- added R19: 0, Resistor_SMD:R_0402_1005Metric_Pad0.72x0.64mm_HandSolder, F.Cu at (-39.8, 29.0)
- added R2: 3.9k, Resistor_SMD:R_0402_1005Metric_Pad0.72x0.64mm_HandSolder, F.Cu at (-45.6, 132.5)
- added R20: 1k, Resistor_SMD:R_0402_1005Metric_Pad0.72x0.64mm_HandSolder, F.Cu at (-40.7, 50.0)
- added R21: 1k, Resistor_SMD:R_0402_1005Metric_Pad0.72x0.64mm_HandSolder, F.Cu at (-40.7, 52.0)
- added R22: 200, Resistor_SMD:R_0402_1005Metric_Pad0.72x0.64mm_HandSolder, F.Cu at (-40.7, 54.0)
- added R23: 1k, Resistor_SMD:R_0402_1005Metric_Pad0.72x0.64mm_HandSolder, F.Cu at (-40.3, 75.0)
- added R24: 1.5k, Resistor_SMD:R_0402_1005Metric_Pad0.72x0.64mm_HandSolder, F.Cu at (-40.3, 77.0)
- added R25: 1.2k, Resistor_SMD:R_0402_1005Metric_Pad0.72x0.64mm_HandSolder, F.Cu at (-40.3, 79.0)
- added R26: 1k, Resistor_SMD:R_0402_1005Metric_Pad0.72x0.64mm_HandSolder, F.Cu at (-39.8, 100.0)
- added R27: 2.7k, Resistor_SMD:R_0402_1005Metric_Pad0.72x0.64mm_HandSolder, F.Cu at (-39.8, 102.0)
- added R28: 6.2k, Resistor_SMD:R_0402_1005Metric_Pad0.72x0.64mm_HandSolder, F.Cu at (-39.8, 104.0)
- added R29: 3.9k, Resistor_SMD:R_0402_1005Metric_Pad0.72x0.64mm_HandSolder, F.Cu at (-15.0, 120.1)
- added R3: 3.9k, Resistor_SMD:R_0402_1005Metric_Pad0.72x0.64mm_HandSolder, F.Cu at (-8.85, 144.0)
- added R30: 1k, Resistor_SMD:R_0402_1005Metric_Pad0.72x0.64mm_HandSolder, F.Cu at (-15.0, 122.1)
- added R31: 1k, Resistor_SMD:R_0402_1005Metric_Pad0.72x0.64mm_HandSolder, F.Cu at (-15.0, 124.1)
- added R32: 1k, Resistor_SMD:R_0402_1005Metric_Pad0.72x0.64mm_HandSolder, F.Cu at (-15.0, 126.0)
- added R33: 3.9k, Resistor_SMD:R_0402_1005Metric_Pad0.72x0.64mm_HandSolder, F.Cu at (36.9, 62.0)
- added R4: 10, Resistor_SMD:R_0402_1005Metric_Pad0.72x0.64mm_HandSolder, F.Cu at (-8.85, 146.0)
- added R5: 3.9k, Resistor_SMD:R_0402_1005Metric_Pad0.72x0.64mm_HandSolder, F.Cu at (-8.85, 148.0)
- added R6: 3.9k, Resistor_SMD:R_0402_1005Metric_Pad0.72x0.64mm_HandSolder, F.Cu at (-8.85, 150.0)
- added R7: 3.9k, Resistor_SMD:R_0402_1005Metric_Pad0.72x0.64mm_HandSolder, F.Cu at (-8.85, 152.0)
- added R8: 3.9k, Resistor_SMD:R_0402_1005Metric_Pad0.72x0.64mm_HandSolder, F.Cu at (27.2, 66.0)
- added R9: 3.9k, Resistor_SMD:R_0402_1005Metric_Pad0.72x0.64mm_HandSolder, F.Cu at (27.2, 68.0)
- added TP1: TestPoint, TestPoint:TestPoint_Pad_D1.0mm, F.Cu at (-11.9, 126.9)
- added TP2: TestPoint, TestPoint:TestPoint_Pad_D1.0mm, F.Cu at (-11.9, 129.9)
- added U1: FT24C256A, Package_SO:MSOP-8_3x3mm_P0.65mm, F.Cu at (-47.9, 127.2)
- added U2: XC7A50T-FGG484, Package_BGA:Xilinx_FGG484, F.Cu at (135.0, 73.0)
- added U3: LP3878MR-ADJ, Package_SO:TI_SO-PowerPAD-8, F.Cu at (-44.6, 3.54)
- added U4: LP3878MR-ADJ, Package_SO:TI_SO-PowerPAD-8, F.Cu at (-44.6, 28.5)
- added U5: LP3878MR-ADJ, Package_SO:TI_SO-PowerPAD-8, F.Cu at (-45.6, 53.5)
- added U6: LP3878MR-ADJ, Package_SO:TI_SO-PowerPAD-8, F.Cu at (-45.2, 78.5)
- added U7: LP3878MR-ADJ, Package_SO:TI_SO-PowerPAD-8, F.Cu at (-44.6, 103.5)
- added U8: MCP23008-E/ML, Package_DFN_QFN:QFN-20-1EP_4x4mm_P0.5mm_EP2.7x2.7mm, F.Cu at (-10.3, 122.2)
- added X1: 50MHz, Oscillator:Oscillator_SMD_Abracon_ASV-4Pin_7.0x5.1mm, F.Cu at (-47.5, 150.5)
Connections:
- net +3V3 renamed Net-(J1-Pin_1)
- J1 pad 10: /GPIO15/RXD0 -> /Raspberry Pi 5/GPIO15/RXD0
- J1 pad 11: /GPIO17 -> /Raspberry Pi 5/GPIO17
- J1 pad 12: /GPIO18/PCM.CLK -> /Raspberry Pi 5/GPIO18/PCM.CLK
- J1 pad 13: /GPIO27 -> /Raspberry Pi 5/GPIO27
- J1 pad 15: /GPIO22 -> /Raspberry Pi 5/GPIO22
- J1 pad 16: /GPIO23 -> /Raspberry Pi 5/GPIO23
- J1 pad 18: /GPIO24 -> /Raspberry Pi 5/GPIO24
- J1 pad 19: /GPIO10/SPI0.MOSI -> /Raspberry Pi 5/GPIO10/SPI0.MOSI
- J1 pad 21: /GPIO9/SPI0.MISO -> /Raspberry Pi 5/GPIO9/SPI0.MISO
- J1 pad 22: /GPIO25 -> /Raspberry Pi 5/GPIO25
- J1 pad 23: /GPIO11/SPI0.SCLK -> /Raspberry Pi 5/GPIO11/SPI0.SCLK
- J1 pad 24: /GPIO8/SPI0.CE0 -> /Raspberry Pi 5/GPIO8/SPI0.CE0
- J1 pad 26: /GPIO7/SPI0.CE1 -> /Raspberry Pi 5/GPIO7/SPI0.CE1
- J1 pad 27: /ID_SDA -> /Raspberry Pi 5/ID_SDA
- J1 pad 28: /ID_SCL -> /Raspberry Pi 5/ID_SCL
- J1 pad 29: /GPIO5 -> /Raspberry Pi 5/GPIO5
- J1 pad 3: /GPIO2/SDA1 -> /Raspberry Pi 5/GPIO2/SDA1
- J1 pad 31: /GPIO6 -> /Raspberry Pi 5/GPIO6
- J1 pad 32: /GPIO12/PWM0 -> /Raspberry Pi 5/GPIO12/PWM0
- J1 pad 33: /GPIO13/PWM1 -> /Raspberry Pi 5/GPIO13/PWM1
- J1 pad 35: /GPIO19/PCM.FS -> /Raspberry Pi 5/GPIO19/PCM.FS
- J1 pad 36: /GPIO16 -> /Raspberry Pi 5/GPIO16
- J1 pad 37: /GPIO26 -> /Raspberry Pi 5/GPIO26
- J1 pad 38: /GPIO20/PCM.DIN -> /Raspberry Pi 5/GPIO20/PCM.DIN
- J1 pad 40: /GPIO21/PCM.DOUT -> /Raspberry Pi 5/GPIO21/PCM.DOUT
- J1 pad 5: /GPIO3/SCL1 -> /Raspberry Pi 5/GPIO3/SCL1
- J1 pad 7: /GPIO4/GPCLK0 -> /Raspberry Pi 5/GPIO4/GPCLK0
- J1 pad 8: /GPIO14/TXD0 -> /Raspberry Pi 5/GPIO14/TXD0
Other:
- board size 65 x 56 mm -> 65 x 53 mm
- copper layers 2 -> 4
- board text removed: "CAMERA (OPTIONAL)"
- board text removed: "DISPLAY (OPTIONAL)"
- board text removed: "Extend PCB edge 0.5mm if using SMT header"
- board text removed: "PoE"

Commit message: Changed linear PSU for SMPS and a few other changes
Parts:
- removed C100, C95, C97, C98, C99: 100u, Capacitor_SMD:C_1206_3216Metric_Pad1.33x1.80mm_HandSolder
- removed C21, C22, C23, C25, C27, C28, C29, C30, C32, C34, C35, C36, C37, C39, C41, C42, C43, C44, C46: 4.7u, Capacitor_SMD:C_0402_1005Metric_Pad0.74x0.62mm_HandSolder
- removed C24: 4.7n, Capacitor_SMD:C_0402_1005Metric_Pad0.74x0.62mm_HandSolder
- removed C31: 3.3n, Capacitor_SMD:C_0402_1005Metric_Pad0.74x0.62mm_HandSolder
- removed C38: 1.5n, Capacitor_SMD:C_0402_1005Metric_Pad0.74x0.62mm_HandSolder
- removed C45: 2.7n, Capacitor_SMD:C_0402_1005Metric_Pad0.74x0.62mm_HandSolder
- removed C49, C50, C51, C52, C53: 10n, Capacitor_SMD:C_0402_1005Metric_Pad0.74x0.62mm_HandSolder
- removed JP1, JP2, JP3, JP4, JP5, JP6: ID_WP, Jumper:SolderJumper-2_P1.3mm_Open_TrianglePad1.0x1.5mm
- removed R16, R17, R20, R21, R23, R26: 1k, Resistor_SMD:R_0402_1005Metric_Pad0.72x0.64mm_HandSolder
- removed R18: 4.99k, Resistor_SMD:R_0402_1005Metric_Pad0.72x0.64mm_HandSolder
- removed R19: 0, Resistor_SMD:R_0402_1005Metric_Pad0.72x0.64mm_HandSolder
- removed R22: 200, Resistor_SMD:R_0402_1005Metric_Pad0.72x0.64mm_HandSolder
- removed R24: 1.5k, Resistor_SMD:R_0402_1005Metric_Pad0.72x0.64mm_HandSolder
- removed R25: 1.2k, Resistor_SMD:R_0402_1005Metric_Pad0.72x0.64mm_HandSolder
- removed R27: 2.7k, Resistor_SMD:R_0402_1005Metric_Pad0.72x0.64mm_HandSolder
- removed R28: 6.2k, Resistor_SMD:R_0402_1005Metric_Pad0.72x0.64mm_HandSolder
- removed U3, U4, U5, U6, U7: LP3878MR-ADJ, Package_SO:TI_SO-PowerPAD-8
- added C101: 22u, Capacitor_SMD:C_0805_2012Metric, F.Cu at (111.3, 97.2)
- added C102: 22u, Capacitor_SMD:C_0805_2012Metric, F.Cu at (123.8, 97.2)
- added C103: 22u, Capacitor_SMD:C_0805_2012Metric, F.Cu at (136.4, 97.2)
- added C104: 22u, Capacitor_SMD:C_0805_2012Metric, F.Cu at (149.1, 97.2)
- added C105: 22u, Capacitor_SMD:C_0805_2012Metric, F.Cu at (102.0, 88.0)
- added C106: 22u, Capacitor_SMD:C_0805_2012Metric, F.Cu at (102.0, 90.0)
- added C107: 4.7u, Capacitor_SMD:C_0402_1005Metric_Pad0.74x0.62mm_HandSolder, F.Cu at (105.2, 86.0)
- added C108: 100n, Capacitor_SMD:C_0402_1005Metric, F.Cu at (118.0, 95.8)
- added C109: 100n, Capacitor_SMD:C_0402_1005Metric, F.Cu at (130.5, 95.8)
- added C110: 100n, Capacitor_SMD:C_0402_1005Metric, F.Cu at (143.1, 95.7)
- added C111: 100n, Capacitor_SMD:C_0402_1005Metric, F.Cu at (155.8, 95.7)
- added C112: 100n, Capacitor_SMD:C_0402_1005Metric_Pad0.74x0.62mm_HandSolder, F.Cu at (105.2, 87.2)
- added C113: 100n, Capacitor_SMD:C_0402_1005Metric_Pad0.74x0.62mm_HandSolder, F.Cu at (105.2, 88.5)
- added C114: 22u, Capacitor_SMD:C_0805_2012Metric, F.Cu at (110.8, 94.2)
- added C115: 22u, Capacitor_SMD:C_0805_2012Metric, F.Cu at (123.2, 94.1)
- added C116: 22u, Capacitor_SMD:C_0805_2012Metric, F.Cu at (133.6, 94.2)
- added C117: 22u, Capacitor_SMD:C_0805_2012Metric, F.Cu at (148.5, 94.2)
- added C118: 22u, Capacitor_SMD:C_0805_2012Metric, F.Cu at (108.5, 94.2)
- added C119: 22u, Capacitor_SMD:C_0805_2012Metric, F.Cu at (121.0, 94.1)
- added C120: 22u, Capacitor_SMD:C_0805_2012Metric, F.Cu at (135.8, 94.2)
- added C121: 22u, Capacitor_SMD:C_0805_2012Metric, F.Cu at (146.2, 94.2)
- added FB4: 600Ω@100MHz, Inductor_SMD:L_0603_1608Metric_Pad1.05x0.95mm_HandSolder, F.Cu at (105.6, 90.0)
- added JP10: ID_WP, Jumper:SolderJumper-2_P1.3mm_Open_TrianglePad1.0x1.5mm, F.Cu at (123.0, 90.8)
- added JP11: ID_WP, Jumper:SolderJumper-2_P1.3mm_Open_TrianglePad1.0x1.5mm, F.Cu at (135.6, 90.8)
- added JP12: ID_WP, Jumper:SolderJumper-2_P1.3mm_Open_TrianglePad1.0x1.5mm, F.Cu at (148.2, 90.7)
- added JP8: ID_WP, Jumper:SolderJumper-2_P1.3mm_Open_TrianglePad1.0x1.5mm, F.Cu at (110.5, 87.0)
- added JP9: ID_WP, Jumper:SolderJumper-2_P1.3mm_Open_TrianglePad1.0x1.5mm, F.Cu at (110.5, 90.8)
- added L1: 4.7u, Inductor_SMD:L_Chilisin_BMRB00050518, F.Cu at (115.2, 91.8)
- added L2: 4.7u, Inductor_SMD:L_Chilisin_BMRB00050518, F.Cu at (127.8, 91.8)
- added L3: 4.7u, Inductor_SMD:L_Chilisin_BMRB00050518, F.Cu at (140.3, 91.8)
- added L4: 4.7u, Inductor_SMD:L_Chilisin_BMRB00050518, F.Cu at (152.9, 91.8)
- added R34: 3.2k, Resistor_SMD:R_0402_1005Metric, F.Cu at (118.5, 98.5)
- added R35: 10k, Resistor_SMD:R_0402_1005Metric, F.Cu at (116.5, 99.0)
- added R36: 5.76k, Resistor_SMD:R_0402_1005Metric, F.Cu at (131.2, 98.5)
- added R37: 10k, Resistor_SMD:R_0402_1005Metric, F.Cu at (129.0, 99.0)
- added R38: 13.7k, Resistor_SMD:R_0402_1005Metric, F.Cu at (144.0, 98.5)
- added R39: 10k, Resistor_SMD:R_0402_1005Metric, F.Cu at (141.7, 99.0)
- added R40: 33.2k, Resistor_SMD:R_0402_1005Metric, F.Cu at (156.5, 98.5)
- added R41: 10k, Resistor_SMD:R_0402_1005Metric, F.Cu at (154.5, 99.0)
- added U10: AP62200TWU-7, Package_TO_SOT_SMD:TSOT-23-6, F.Cu at (127.9, 96.7)
- added U11: AP62200TWU-7, Package_TO_SOT_SMD:TSOT-23-6, F.Cu at (140.5, 96.7)
- added U12: AP62200TWU-7, Package_TO_SOT_SMD:TSOT-23-6, F.Cu at (153.1, 96.7)
- added U9: AP62200TWU-7, Package_TO_SOT_SMD:TSOT-23-6, F.Cu at (115.4, 96.7)
- C14, C16, C17, C20: value 4.7u -> 22n; footprint Capacitor_SMD:C_0402_1005Metric_Pad0.74x0.62mm_HandSolder -> Capacitor_SMD:C_0402_1005Metric
- C18: value 4.7n -> 10n; footprint Capacitor_SMD:C_0402_1005Metric_Pad0.74x0.62mm_HandSolder -> Capacitor_SMD:C_0402_1005Metric
- C8: value 4.7u -> 100u; footprint Capacitor_SMD:C_0402_1005Metric_Pad0.74x0.62mm_HandSolder -> Capacitor_SMD:C_1206_3216Metric_Pad1.33x1.80mm_HandSolder
- C9: value 4.7u -> 10n; footprint Capacitor_SMD:C_0402_1005Metric_Pad0.74x0.62mm_HandSolder -> Capacitor_SMD:C_0402_1005Metric
- D1: footprint LED_SMD:LED_0603_1608Metric_Pad1.05x0.95mm_HandSolder -> LED_SMD:LED_0402_1005Metric
- R14: value 0 -> 45k; footprint Resistor_SMD:R_0402_1005Metric_Pad0.72x0.64mm_HandSolder -> Resistor_SMD:R_0402_1005Metric
- R15: value 4.99k -> 10k; footprint Resistor_SMD:R_0402_1005Metric_Pad0.72x0.64mm_HandSolder -> Resistor_SMD:R_0402_1005Metric
- moved C1 229.4 mm to (167.5, 61.3)
- moved R1 229.4 mm to (171.9, 57.7)
- moved R2 229.4 mm to (171.9, 59.7)
- moved U1 229.4 mm to (169.6, 54.5)
- moved C16 225.1 mm to (157.0, 95.8), turned to 90 degrees
- moved C20 218.2 mm to (156.5, 97.2)
- moved C14 214.6 mm to (144.5, 95.8), turned to 90 degrees
- moved C18 212.2 mm to (144.0, 97.2)
- moved C17 201.6 mm to (131.2, 97.2)
- moved C9 193.1 mm to (118.5, 97.2)
- moved JP7 156.8 mm to (108.7, 51.5)
- moved R14 45.8 mm to (-85.5, -0.99)
- moved R15 45.8 mm to (-85.5, 1.00)
- moved R11 34.8 mm to (104.0, 62.5), turned to 180 degrees
- moved D1 31.3 mm to (101.5, 62.5)
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Connections:
- C14 pad 1: GND -> /FPGA Top/FPGA Power/SEQ3
- C14 pad 2: Net-(JP2-B) -> GND
- C16 pad 1: GND -> /FPGA Top/FPGA Power/SEQ4
- C16 pad 2: Net-(JP2-B) -> GND
- C17 pad 1: GND -> /FPGA Top/FPGA Power/SEQ2
- C17 pad 2: Net-(JP2-B) -> GND
- C18 pad 1: Net-(U3-ADJ) -> /FPGA Top/FPGA Power/SEQ3
- C18 pad 2: Net-(JP2-B) -> GND
- C20 pad 1: GND -> /FPGA Top/FPGA Power/SEQ4
- C20 pad 2: +5V -> GND
- C9 pad 1: GND -> /FPGA Top/FPGA Power/SEQ1
- C9 pad 2: +5V -> GND
- R14 pad 1: Net-(U3-ADJ) -> Net-(U2F-VP_0)
- R14 pad 2: Net-(JP2-B) -> +5V
- R15 pad 2: Net-(U3-ADJ) -> Net-(U2F-VP_0)
- U2 pad L10: GND -> Net-(U2F-VP_0)
Routing:
- net GND: track 0.00 -> 32.8 mm
- net /FPGA Top/FPGA Power/SEQ3: track 0.00 -> 3.72 mm
- net /FPGA Top/FPGA Power/SEQ4: track 0.00 -> 3.41 mm
- net /FPGA Top/FPGA Power/SEQ2: track 0.00 -> 2.00 mm
- net /FPGA Top/FPGA Power/SEQ1: track 0.00 -> 1.74 mm
- net Net-(U9-BST): track 0.00 -> 1.71 mm
- net Net-(U10-BST): track 0.00 -> 1.70 mm
- net Net-(U12-BST): track 0.00 -> 1.69 mm
- net Net-(U11-BST): track 0.00 -> 1.69 mm
- added copper zone on F.Cu, net +5V
- added copper zone on F.Cu, net GND
- added copper zone on F.Cu, net Net-(JP10-A)
- added copper zone on F.Cu, net Net-(JP11-A)
- added copper zone on F.Cu, net Net-(JP9-A)
- added copper zone on F.Cu, net Net-(U10-FB)
- added copper zone on F.Cu, net Net-(U10-SW)
- added copper zone on F.Cu, net Net-(U11-FB)
- added copper zone on F.Cu, net Net-(U11-SW)
- added copper zone on F.Cu, net Net-(U12-FB)
- added copper zone on F.Cu, net Net-(U12-SW)
- added copper zone on F.Cu, net Net-(U9-FB)
- added copper zone on F.Cu, net Net-(U9-SW)
Other:
- board text added: "1V0"
- board text added: "1V2MGT"
- board text added: "1V8"
- board text added: "3V3"
- board text added: "MGT"
- board text removed: "RJ45"
- board text removed: "USB"

Commit message: Started routing. More to go
Parts:
- removed C47: 100n, Capacitor_SMD:C_0402_1005Metric_Pad0.74x0.62mm_HandSolder
- removed C48: 4.7u, Capacitor_SMD:C_0402_1005Metric_Pad0.74x0.62mm_HandSolder
- removed D2: RED, LED_SMD:LED_0603_1608Metric_Pad1.05x0.95mm_HandSolder
- removed JP7: ID_WP, Jumper:SolderJumper-2_P1.3mm_Open_TrianglePad1.0x1.5mm
- removed R29, R33: 3.9k, Resistor_SMD:R_0402_1005Metric_Pad0.72x0.64mm_HandSolder
- removed R30, R31, R32: 1k, Resistor_SMD:R_0402_1005Metric_Pad0.72x0.64mm_HandSolder
- removed TP2: TestPoint, TestPoint:TestPoint_Pad_D1.0mm
- removed U8: MCP23008-E/ML, Package_DFN_QFN:QFN-20-1EP_4x4mm_P0.5mm_EP2.7x2.7mm
- added R16: 10, Resistor_SMD:R_0402_1005Metric_Pad0.72x0.64mm_HandSolder, F.Cu at (154.9, 69.5)
- added R17: 3.9k, Resistor_SMD:R_0402_1005Metric_Pad0.72x0.64mm_HandSolder, F.Cu at (120.1, 76.0)
- TP1: value TestPoint -> 50M
- moved FB3 232.1 mm to (162.1, 60.8)
- moved C94 229.0 mm to (162.4, 62.2)
- moved C93 227.7 mm to (162.4, 63.5)
- moved X1 223.9 mm to (160.5, 67.5), turned to 180 degrees
- moved R14 213.3 mm to (113.5, 75.8), turned to 180 degrees
- moved R15 212.9 mm to (113.5, 76.8)
- moved J2 186.7 mm to (162.8, 86.5), turned to 180 degrees
- moved C96 183.8 mm to (115.1, 79.0), turned to 180 degrees
- moved R6 180.6 mm to (157.2, 79.1), turned to 90 degrees
- moved R5 180.2 mm to (158.5, 81.1), turned to 90 degrees
- moved R7 179.8 mm to (157.2, 83.2), turned to -90 degrees
- moved R3 177.4 mm to (158.5, 85.1), turned to 90 degrees
- moved R4 176.2 mm to (157.2, 87.1), turned to -90 degrees
- moved TP1 174.1 mm to (152.5, 69.5)
- moved C8 166.6 mm to (103.4, 52.8)
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Connections:
- net Net-(C10-Pad2) renamed /FPGA Top/FPGA Bank 216 (MGT)/MGTAVTT
- net Net-(C11-Pad2) renamed /FPGA Top/FPGA Bank 216 (MGT)/MGTAVCC
- net Net-(U2F-VP_0) renamed /FPGA Top/FPGA Config/5V_SNS
- C1 pad 1: GND -> +3.3VP
- C1 pad 2: +3V3 -> GND
- J1 pad 1: Net-(J1-Pin_1) -> +3.3VP
- J1 pad 17: Net-(J1-Pin_1) -> +3.3VP
- R1 pad 1: +3V3 -> +3.3VP
- R2 pad 1: +3V3 -> +3.3VP
- R3 pad 1: Net-(J2-Pin_2) -> +3V3
- R5 pad 1: Net-(J2-Pin_2) -> +3V3
- R6 pad 1: Net-(J2-Pin_2) -> +3V3
- TP1 pad 1: Net-(U8-GP5) -> /FPGA Top/CLK50MHZ
- U1 pad 1: unconnected-(U1-A0-Pad1) -> GND
- U1 pad 2: unconnected-(U1-A1-Pad2) -> GND
- U1 pad 3: unconnected-(U1-A2-Pad3) -> GND
- U1 pad 7: Net-(JP1-A) -> GND
- U1 pad 8: +3V3 -> +3.3VP
- U2 pad A16: unconnected-(U2B-IO_L9N_T1_DQS_16-PadA16) -> /Raspberry Pi 5/GPIO5
- U2 pad A18: unconnected-(U2B-IO_L17P_T2_16-PadA18) -> /Raspberry Pi 5/GPIO6
- U2 pad A19: unconnected-(U2B-IO_L17N_T2_16-PadA19) -> /Raspberry Pi 5/GPIO12/PWM0
- U2 pad A21: unconnected-(U2B-IO_L21N_T3_DQS_16-PadA21) -> /Raspberry Pi 5/GPIO13/PWM1
- U2 pad B1: /Raspberry Pi 5/GPIO14/TXD0 -> /Raspberry Pi 5/GPIO18/PCM.CLK
- U2 pad B2: unconnected-(U2C-IO_L2N_T0_AD12N_35-PadB2) -> /Raspberry Pi 5/GPIO27
- U2 pad B20: unconnected-(U2B-IO_L16P_T2_16-PadB20) -> /Raspberry Pi 5/GPIO16
- U2 pad C2: /Raspberry Pi 5/GPIO15/RXD0 -> unconnected-(U2C-IO_L2P_T0_AD12P_35-PadC2)
- U2 pad C22: unconnected-(U2B-IO_L20P_T3_16-PadC22) -> /Raspberry Pi 5/GPIO26
- U2 pad D1: unconnected-(U2C-IO_L3N_T0_DQS_AD5N_35-PadD1) -> /Raspberry Pi 5/GPIO17
- U2 pad D17: unconnected-(U2B-IO_L12P_T1_MRCC_16-PadD17) -> /Raspberry Pi 5/GPIO21/PCM.DOUT
- U2 pad D19: unconnected-(U2B-IO_L14N_T2_SRCC_16-PadD19) -> /Raspberry Pi 5/GPIO20/PCM.DIN
- U2 pad E1: unconnected-(U2C-IO_L3P_T0_DQS_AD5P_35-PadE1) -> /Raspberry Pi 5/GPIO15/RXD0
- U2 pad E19: unconnected-(U2B-IO_L14P_T2_SRCC_16-PadE19) -> /Raspberry Pi 5/GPIO19/PCM.FS
- U2 pad E2: /FPGA Top/PCIE_DET_WAKE -> unconnected-(U2C-IO_L4P_T0_35-PadE2)
- U2 pad F1: unconnected-(U2C-IO_L5N_T0_AD13N_35-PadF1) -> /Raspberry Pi 5/GPIO4/GPCLK0
- U2 pad F3: Net-(U2C-IO_L6P_T0_35) -> /Raspberry Pi 5/GPIO22
- U2 pad G1: /FPGA Top/PCIE_CLKREQ_N -> /FPGA Top/PCIE_RST_B
- U2 pad G4: /Raspberry Pi 5/GPIO21/PCM.DOUT -> unconnected-(U2C-IO_L12N_T1_MRCC_35-PadG4)
- U2 pad H4: /FPGA Top/CLK50MHZ -> unconnected-(U2C-IO_L12P_T1_MRCC_35-PadH4)
- U2 pad J1: /FPGA Top/PCIE_RST_B -> /FPGA Top/PCIE_CLKREQ_N
- U2 pad J19: unconnected-(U2B-IO_L12P_T1_MRCC_15-PadJ19) -> /FPGA Top/CLK50MHZ
- U2 pad J4: /Raspberry Pi 5/GPIO20/PCM.DIN -> unconnected-(U2C-IO_L13N_T2_MRCC_35-PadJ4)
- U2 pad J6: /Raspberry Pi 5/GPIO13/PWM1 -> unconnected-(U2C-IO_L17N_T2_35-PadJ6)
- U2 pad K1: unconnected-(U2C-IO_L7P_T1_AD6P_35-PadK1) -> /FPGA Top/PCIE_DET_WAKE
- U2 pad K3: /Raspberry Pi 5/GPIO17 -> unconnected-(U2C-IO_L14N_T2_SRCC_35-PadK3)
- U2 pad K4: /Raspberry Pi 5/GPIO19/PCM.FS -> unconnected-(U2C-IO_L13P_T2_MRCC_35-PadK4)
- U2 pad K6: /Raspberry Pi 5/GPIO12/PWM0 -> unconnected-(U2C-IO_L17P_T2_35-PadK6)
- U2 pad L1: /Raspberry Pi 5/GPIO4/GPCLK0 -> /Raspberry Pi 5/GPIO14/TXD0
- U2 pad L3: /Raspberry Pi 5/GPIO18/PCM.CLK -> unconnected-(U2C-IO_L14P_T2_SRCC_35-PadL3)
- U2 pad L4: /Raspberry Pi 5/GPIO26 -> unconnected-(U2C-IO_L18N_T2_35-PadL4)
- U2 pad L5: /Raspberry Pi 5/GPIO22 -> unconnected-(U2C-IO_L18P_T2_35-PadL5)
- U2 pad M1: /Raspberry Pi 5/GPIO16 -> /Raspberry Pi 5/GPIO3/SCL1
- U2 pad M2: /Raspberry Pi 5/GPIO6 -> unconnected-(U2C-IO_L16N_T2_35-PadM2)
- U2 pad M3: /Raspberry Pi 5/GPIO5 -> unconnected-(U2C-IO_L16P_T2_35-PadM3)
- U2 pad N4: /Raspberry Pi 5/GPIO27 -> unconnected-(U2C-IO_L19P_T3_35-PadN4)
- U2 pad P1: unconnected-(U2C-IO_L20N_T3_35-PadP1) -> /Raspberry Pi 5/GPIO2/SDA1
- U2 pad R1: unconnected-(U2C-IO_L20P_T3_35-PadR1) -> Net-(U2C-IO_L20P_T3_35)
- X1 pad 3: /FPGA Top/CLK50MHZ -> Net-(X1-OUT)
Routing:
- net GND: track 32.8 -> 99.3 mm, vias 0 -> 142
- net /Raspberry Pi 5/GPIO23: track 0.00 -> 52.7 mm, vias 0 -> 3
- net /Raspberry Pi 5/GPIO10/SPI0.MOSI: track 0.00 -> 46.4 mm, vias 0 -> 1
- net +3.3VP: track 0.00 -> 45.9 mm, vias 0 -> 1
- net /Raspberry Pi 5/GPIO24: track 0.00 -> 37.8 mm, vias 0 -> 2
- net /Raspberry Pi 5/GPIO8/SPI0.CE0: track 0.00 -> 37.7 mm, vias 0 -> 1
- net /Raspberry Pi 5/GPIO11/SPI0.SCLK: track 0.00 -> 37.7 mm, vias 0 -> 2
- net /Raspberry Pi 5/GPIO7/SPI0.CE1: track 0.00 -> 37.1 mm, vias 0 -> 1
- net /Raspberry Pi 5/GPIO9/SPI0.MISO: track 0.00 -> 36.6 mm, vias 0 -> 2
- net TCK: track 0.00 -> 35.4 mm, vias 0 -> 1
- net /Raspberry Pi 5/GPIO2/SDA1: track 0.00 -> 32.6 mm
- net +3V3: track 0.00 -> 31.3 mm, vias 0 -> 41
- net /Raspberry Pi 5/GPIO14/TXD0: track 0.00 -> 31.1 mm
- net /Raspberry Pi 5/GPIO25: track 0.00 -> 30.7 mm, vias 0 -> 2
- net TDO: track 0.00 -> 30.2 mm, vias 0 -> 1
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- added copper zone on In1.Cu, net GND
Other:
- board size 65 x 53 mm -> 65 x 56 mm

Commit message: More routing and tinkering. Need to do non-MGT decoupling next.
Parts:
- removed C13, C19, C33, C40, C55, C56, C57, C58, C59, C60, C61, C62, C63, C64, C66, C67, C68, C69, C70, C72, C73, C74, C75, C76, C77, C79, C80, C81, C82, C83, C84, C86, C87, C88, C89, C90, C91: 100n, Capacitor_SMD:C_0402_1005Metric_Pad0.74x0.62mm_HandSolder
- removed C26, C54, C65, C71, C78, C85, C92: 4.7u, Capacitor_SMD:C_0402_1005Metric_Pad0.74x0.62mm_HandSolder
- added C21: 100n, Capacitor_SMD:C_0402_1005Metric_Pad0.74x0.62mm_HandSolder, F.Cu at (157.9, 76.5)
- C10, C11, C12, C15, C4, C5: moved to B.Cu
- moved C10 52.4 mm to (133.6, 60.0), turned to 180 degrees
- moved C4 51.9 mm to (135.1, 63.0), turned to 180 degrees
- moved C11 51.7 mm to (133.5, 63.9), turned to -90 degrees
- moved C12 47.7 mm to (128.5, 63.9), turned to -90 degrees
- moved R13 47.4 mm to (130.4, 58.7), turned to 180 degrees
- moved C5 44.1 mm to (126.5, 63.0)
- moved FB2 43.2 mm to (127.5, 59.0), turned to 180 degrees
- moved C15 40.2 mm to (121.8, 69.1), turned to 90 degrees
- moved FB1 31.8 mm to (119.9, 72.2), turned to 90 degrees
- moved R9 8.73 mm to (137.4, 58.1), turned to 180 degrees
- moved R8 7.90 mm to (137.4, 59.2), turned to 180 degrees
- moved JP8 5.13 mm to (105.5, 86.5), turned to 0 degrees
- moved C107 3.72 mm to (102.7, 88.2), turned to 0 degrees
- moved C113 3.36 mm to (102.7, 85.8), turned to 0 degrees
- moved C112 2.51 mm to (102.7, 87.0), turned to 0 degrees
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Connections:
- net +1V2 renamed +1V2_MGTAVTT
- net Net-(JP8-A) renamed /FPGA Top/FPGA Power/1V0_FB
- net Net-(U2E-MGTRREF_216) renamed /FPGA Top/FPGA Bank 216 (MGT)/MR
- FB1 pad 1: +1V0 -> +1V0_MGTAVCC
- JP8 pad 2: +1V0 -> +1V0_MGTAVCC
- U2 pad B16: unconnected-(U2B-IO_L7N_T1_16-PadB16) -> /Raspberry Pi 5/GPIO8/SPI0.CE0
- U2 pad B17: unconnected-(U2B-IO_L11P_T1_SRCC_16-PadB17) -> /Raspberry Pi 5/GPIO7/SPI0.CE1
- U2 pad W19: /Raspberry Pi 5/GPIO8/SPI0.CE0 -> unconnected-(U2A-IO_L12P_T1_MRCC_14-PadW19)
- U2 pad W20: /Raspberry Pi 5/GPIO7/SPI0.CE1 -> unconnected-(U2A-IO_L12N_T1_MRCC_14-PadW20)
Routing:
- net +3V3: track 31.3 -> 111.5 mm, vias 41 -> 54
- net +1V2_MGTAVTT: track 0.00 -> 39.8 mm, vias 0 -> 3
- net +1V0: track 12.0 -> 43.0 mm, vias 17 -> 19
- net +1V0_MGTAVCC: track 0.00 -> 23.2 mm
- net /FPGA Top/FPGA Bank 216 (MGT)/MGTAVCC: track 3.54 -> 26.4 mm, vias 5 -> 7
- net GND: track 99.3 -> 121.0 mm, vias 142 -> 194
- net /Raspberry Pi 5/GPIO7/SPI0.CE1: track 37.1 -> 17.9 mm
- net /FPGA Top/FPGA Bank 216 (MGT)/MGTAVTT: track 4.24 -> 22.8 mm, vias 6 -> 8
- net /Raspberry Pi 5/GPIO8/SPI0.CE0: track 37.7 -> 20.0 mm
- net +1V8: track 4.95 -> 18.7 mm, vias 7 -> 9
- net Net-(JP11-A): track 0.00 -> 9.76 mm, vias 0 -> 2
- net Net-(JP10-A): track 0.00 -> 9.76 mm, vias 0 -> 2
- net Net-(JP12-A): track 0.00 -> 9.75 mm, vias 0 -> 2
- net Net-(JP9-A): track 0.00 -> 9.75 mm, vias 0 -> 2
- net /FPGA Top/FPGA Bank 216 (MGT)/MR: track 0.71 -> 8.62 mm, vias 1 -> 2
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- added copper zone on In2.Cu, net +1V0
- added copper zone on B.Cu, net +1V8
- added copper zone on B.Cu, net +3V3
- added copper zone on B.Cu, net +5V
- added copper zone on F.Cu, net /FPGA Top/FPGA Power/1V0_FB
- added copper zone on F.Cu, net Net-(JP12-A)
Other:
- board text added: "1V2"
- board text added: "MGTAVCC"
- board text added: "MGTAVTT"
- board text added: "VCCAUX/BAT"
- board text added: "VCCINT/BRAM"
- board text added: "VCCO"
- board text removed: "1V2MGT"
- board text removed: "MGT"
